Commit message: 22:56

File: install/example_description/share/example_description/robot/visual/my-robot.xacro (robot description, xacro)
@@ -28,5 +28,5 @@
   <link name="link_2">
     <visual>
-      <origin xyz="0.0 0.0 0.0" rpy="0 0 ${-3.14/2}"/>
+      <origin xyz="0.0 0.0 0.0" rpy="0 0 0"/>
       <geometry>
         <mesh filename="file:///$(find example_description)/meshes/link_2.stl"/>
@@ -37,5 +37,5 @@
     <parent link="link_1"/>
     <child link="link_2"/>
-    <origin xyz="0.0 -0.12 0.0" rpy="${-3.14/2} 0 0"/>
+    <origin xyz="0.0 -0.12 0.0" rpy="${-3.14/2} ${-3.14/2} 0"/>
     <axis xyz="0 0 1"/>
     <limit
@@ -47,5 +47,5 @@
   <link name="link_3">
     <visual>
-      <origin xyz="0.0 0.0 0.0" rpy="0 0 ${-3.14/2}"/>
+      <origin xyz="0.0 0.0 0.0" rpy="0 0 0"/>
       <geometry>
         <mesh filename="file:///$(find example_description)/meshes/link_3.stl"/>
@@ -56,5 +56,5 @@
     <parent link="link_2"/>
     <child link="link_3"/>
-    <origin xyz="0.0 -0.25 0.1" rpy="0 0 0"/>
+    <origin xyz="0.25 0.0 0.1" rpy="0 0 0"/>
     <axis xyz="0 0 1"/>
     <limit
@@ -75,5 +75,5 @@
     <parent link="link_3"/>
     <child link="end_effector"/>
-    <origin xyz="0.0 -0.28 0.0" rpy="${3.14/2} 0 0"/>
+    <origin xyz="0.28 0.0 0.0" rpy="${3.14/2} 0 ${3.14/2}"/>
   </joint>
 </robot>

Commit message: 19:27

File: install/example_description/share/example_description/robot/visual/my-robot.xacro (robot description, xacro)
@@ -3,6 +3,7 @@
   <link name="link_0">
     <visual>
+      <origin rpy="0 0 0" xyz="0 0 0"/>
       <geometry>
-        <mesh filename="file:///$(find example_description)/meshes/link_0.stl"/>
+        <mesh filename="package://example_description/meshes/link_0.stl"/>
       </geometry>
     </visual>
@@ -10,63 +11,52 @@
   <link name="link_1">
     <visual>
+      <origin rpy="0 0 0" xyz="0 0 0"/>
       <geometry>
-        <mesh filename="file:///$(find example_description)/meshes/link_1.stl"/>
+        <mesh filename="package://example_description/meshes/link_1.stl"/>
       </geometry>
     </visual>
   </link>
   <joint name="joint_1" type="revolute">
+    <axis xyz="0 0 1"/>
+    <limit effort="1000.0" lower="-3.14159265359" upper="3.14159265359" velocity="0.5"/>
+    <origin rpy="0 0 0" xyz="0 0 0.2"/>
     <parent link="link_0"/>
     <child link="link_1"/>
-    <origin xyz="0 0 0.2" rpy="0 0 0"/>
-    <axis xyz="0 0 1"/>
-    <limit
-      lower="-3.1459"
-      upper="3.1459"
-      velocity="1000.0"
-      effort="1000.0"/>
   </joint>
   <link name="link_2">
     <visual>
-      <origin xyz="0.0 0.0 0.0" rpy="0 0 0"/>
+      <origin rpy="0 0 0" xyz="0 0 0"/>
       <geometry>
-        <mesh filename="file:///$(find example_description)/meshes/link_2.stl"/>
+        <mesh filename="package://example_description/meshes/link_2.stl"/>
       </geometry>
     </visual>
   </link>
   <joint name="joint_2" type="revolute">
+    <axis xyz="0 0 1"/>
+    <limit effort="1000.0" lower="-3.14159265359" upper="3.14159265359" velocity="0.5"/>
+    <origin rpy="-1.57 -1.57 0" xyz="0 -0.12 0" />
     <parent link="link_1"/>
     <child link="link_2"/>
-    <origin xyz="0.0 -0.12 0.0" rpy="${-3.14/2} ${-3.14/2} 0"/>
-    <axis xyz="0 0 1"/>
-    <limit
-      lower="-3.1459"
-      upper="3.1459"
-      velocity="1000.0"
-      effort="1000.0"/>
   </joint>
   <link name="link_3">
     <visual>
-      <origin xyz="0.0 0.0 0.0" rpy="0 0 0"/>
+      <origin rpy="0 0 0" xyz="0 0 0"/>
       <geometry>
-        <mesh filename="file:///$(find example_description)/meshes/link_3.stl"/>
+        <mesh filename="package://example_description/meshes/link_3.stl"/>
       </geometry>
     </visual>
   </link>
   <joint name="joint_3" type="revolute">
+    <axis xyz="0 0 1"/>
+    <limit effort="1000.0" lower="-3.14159265359" upper="3.14159265359" velocity="0.5"/>
+    <origin rpy="0 0 0" xyz="0.25 0 0.10"/>
     <parent link="link_2"/>
     <child link="link_3"/>
-    <origin xyz="0.25 0.0 0.1" rpy="0 0 0"/>
-    <axis xyz="0 0 1"/>
-    <limit
-      lower="-3.1459"
-      upper="3.1459"
-      velocity="1000.0"
-      effort="1000.0"/>
   </joint>
   <link name="end_effector">
     <visual>
-      <origin xyz="0.0 0.0 0.0" rpy="0 0 0"/>
+      <origin rpy="0 0 0" xyz="0 0 0"/>
       <geometry>
-        <mesh filename="file:///$(find example_description)/meshes/end_effector.stl"/>
+        <mesh filename="package://example_description/meshes/end_effector.stl"/>
       </geometry>
     </visual>
@@ -75,5 +65,5 @@
     <parent link="link_3"/>
     <child link="end_effector"/>
-    <origin xyz="0.28 0.0 0.0" rpy="${3.14/2} 0 ${3.14/2}"/>
+    <origin xyz="0.28 0.0 0.0" rpy="1.57079632679 0 1.57079632679"/>
   </joint>
 </robot>
